Commit message: Inertial Data for links in URDF files, update to gymnasium

File: envs/ur5.urdf (robot description, URDF)
Before this commit: robot ur5, 7 links, 6 joints
Links:
- link base_link: mass None -> 1.0
- link ee_link: mass None -> 0.2
- link link1: mass None -> 0.5
- link link2: mass None -> 0.5
- link link3: mass None -> 0.5
- link link4: mass None -> 0.3
- link link5: mass None -> 0.3
